File: rs232-rs485sniffer/rs232-rs485sniffer.kicad_sch (KiCad schematic)
At the start: 13 parts, among them J1 supply, J2 Conn_01x05_Pin, U1 MAX232, U2 MAX485E, U3 MAX485E, U4 AMS1117-5.0

Commit message: [FIX] Stable version
Parts:
- removed J2: Conn_01x05_Pin, symbol Connector:Conn_01x05_Pin
- removed U3: MAX485E, Package_SO:SOIC-8_3.9x4.9mm_P1.27mm, symbol Interface_UART:MAX485E
- added C5, C6: 100uf, Capacitor_THT:CP_Radial_D8.0mm_P3.80mm, symbol Device:C_Polarized
- added J2: USB_B, Connector_USB:USB_B_Lumberg_2411_02_Horizontal, symbol Connector:USB_B
- added RS485_sniffer1: Conn_01x03_Pin, TerminalBlock_Phoenix:TerminalBlock_Phoenix_MKDS-1,5-3-5.08_1x03_P5.08mm_Horizontal, symbol Connector:Conn_01x03_Pin
- C1, C2, C3, C4: footprint (none) -> Capacitor_THT:CP_Radial_D8.0mm_P3.80mm
- J1: value supply -> supply pin 5 GND pin 9 +12V; footprint (none) -> TerminalBlock_Phoenix:TerminalBlock_Phoenix_MKDS-1,5-2_1x02_P5.00mm_Horizontal
- R1, R2: value 10k -> 1k; footprint (none) -> Inductor_SMD:L_1206_3216Metric_Pad1.22x1.90mm_HandSolder
- ReceiverRS-232: footprint (none) -> TerminalBlock_Phoenix:TerminalBlock_Phoenix_MKDS-1,5-3-5.08_1x03_P5.08mm_Horizontal
- U1: footprint (none) -> Package_DIP:DIP-16_W7.62mm_Socket_LongPads
Connections:
- net +5V: now also C6.1, J2.1 (VBUS); no longer R1.1, R2.1
- net GND: now also C5.2, C6.2, J2.4 (GND), RS485_sniffer1.1 (Pin_1)
- net at U2.1 (RO): no longer R1.2
- net at U2.4 (DI): now also R1.2, R2.2; no longer U1.9 (R2OUT)
- net at U2.6 (A): now also RS485_sniffer1.3 (Pin_3)
- net at U2.7 (B): now also RS485_sniffer1.2 (Pin_2)
- net at J1.1 (Pin_1), U4.3 (VI): now also C5.1
- net at U1.12 (R1OUT): now also R1.1
- new net: R2.1, U1.9 (R2OUT)
